Commit message: step 40 INCOMPLETE

File: body.urdf (robot description, URDF)
Before this commit: robot robot, 3 links, 2 joints
Links:
- added link LeftLeg, mass 1; collision box size=1 0.2 0.2; visual box size=1 0.2 0.2
- added link RightLeg, mass 1; collision box size=0.2 1 0.2; visual box size=0.2 1 0.2
Joints:
- added joint Torso_LeftLeg: type revolute, parent Torso, child LeftLeg, origin xyz=-0.5 0 1 rpy=0 0 0, axis 0 1 0, limit lower=-3.14159 upper=3.14159 effort=0.0 velocity=0.0
- added joint Torso_RightLeg: type revolute, parent Torso, child RightLeg, origin xyz=-0.5 0 0 rpy=0 0 0, axis 0 1 0, limit lower=-3.14159 upper=3.14159 effort=0.0 velocity=0.0
- joint Torso_BackLeg: axis 0 1 0 -> 1 0 0
- joint Torso_FrontLeg: axis 0 1 0 -> 1 0 0

Commit message: step 40 INCOMPLETE

File: body.urdf (robot description, URDF)
Before this commit: robot robot, 5 links, 4 joints
Links:
- link RightLeg: geometry collision box size=1 0.2 0.2; visual box size=1 0.2 0.2
Joints:
- joint Torso_RightLeg: origin xyz=-0.5 0 0 rpy=0 0 0 -> xyz=0.5 0 1 rpy=0 0 0

Commit message: we have a semi functioning camera. and some sleep at the end of the constructor to simulate the connection to the crazyflies.

File: body.urdf (robot description, URDF)
Before this commit: robot robot, 3 links, 2 joints
Links:
- link BackLeg: geometry collision box size=0.5 0.5 0.5; visual box size=0.5 0.5 0.5
- link FrontLeg: geometry collision box size=0.5 0.5 0.5; visual box size=0.5 0.5 0.5
- link Torso: geometry collision box size=0.5 0.5 0.5; visual box size=0.5 0.5 0.5

Commit message: going to try and use a nested synccrazyflie class to do this sime demo

File: body.urdf (robot description, URDF)
Before this commit: robot robot, 3 links, 2 joints
Links:
- link BackLeg: geometry collision box size=1 1 1; visual box size=1 1 1
- link FrontLeg: geometry collision box size=1 1 1; visual box size=1 1 1
- link Torso: geometry collision box size=1 1 1; visual box size=1 1 1
