Commit message: Step 16 added tools to determine the most distance covered, compared quad to hex to octo pod

File: body126.urdf (robot description, URDF)
Before this commit: robot robot, 13 links, 12 joints
Links:
- removed link BackLeftLeg
- removed link BackLeftLowerLeg
- removed link FrontLeftLeg
- removed link FrontLeftLowerLeg
- removed link FrontRightLeg
- removed link FrontRightLowerLeg
- added link LeftLeg, mass 1; collision box size=1 0.2 0.2; visual box size=1 0.2 0.2
- added link LeftLowerLeg, mass 1; collision box size=0.2 0.2 1; visual box size=0.2 0.2 1
- link Torso: geometry collision box size=1 1 1; visual box size=1 1 1
Joints:
- removed joint BackLeftLeg_BackLeftLowerLeg
- removed joint FrontLeftLeg_FrontLeftLowerLeg
- removed joint FrontRightLeg_FrontRightLowerLeg
- removed joint Torso_BackLeftLeg
- removed joint Torso_FrontLeftLeg
- removed joint Torso_FrontRightLeg
- added joint LeftLeg_LeftLowerLeg: type revolute, parent LeftLeg, child LeftLowerLeg, origin xyz=-1 0 0 rpy=0 0 0, axis 0 1 0, limit lower=-3.14159 upper=3.14159 effort=0.0 velocity=0.0
- added joint Torso_LeftLeg: type revolute, parent Torso, child LeftLeg, origin xyz=-0.5 0 1 rpy=0 0 0, axis 0 1 0, limit lower=-3.14159 upper=3.14159 effort=0.0 velocity=0.0
